File: hardware/maus-blenano2-mk-1.0.0.sch (EAGLE design)
At the start: 14 parts, among them Q1 SI2301CDS, U1 REDBEAR_BLE_NANO2_LESS, U2 MCP73831T-2ACI/OT

Commit message: initial rev of ble nano2 daughter board
Parts:
- removed JP1: M05X2SMD_RA, a_parts:M05X2SMD_RA
- added J1: M04X2SMD_RA, a_parts:M04X2SMD_RA
- D1: value (none) -> PMEG2005CT; device a_parts:DIODE-SCHOTTKYSOD123 -> a_parts:DIODE-SCHOTTKY-DUALPMEG2005CT
- JP2: value M02JST-ZH-SM4-VERT-R+ -> M02JST-SH-VERT; device a_parts:M02JST-ZH-SM4-VERT-R+ -> a_parts:M02JST-SH-VERT
- R2: value 10K -> 100K
- renumbered CHG to CHARGE
Connections:
- removed net IRRECV: JP1.2, U1.D3
- net 3.3V: now also J1.3; no longer JP1.5
- net 5V: now also D1.A2; no longer D1.A
- net AIN1: now also J1.6, U1.D3; no longer JP1.7, U1.D0
- net AIN2: now also J1.5, U1.D2; no longer JP1.9, U1.D1
- net BIN1: now also J1.7, U1.D1; no longer JP1.8, U1.D4
- net BIN2: now also J1.8, U1.D0; no longer JP1.10, U1.D5
- net GND: now also J1.1; no longer JP1.3
- net VIN: now also D1.K, J1.2; no longer D1.C, JP1.1
Other:
- moved on the sheet: Q1
