File: hardware/maus-blenano2-mk-1.0.1.brd (EAGLE design)
At the start: 20 x 18 mm, 17 parts, among them M1 M02JST-SH-VERT, M2 M02JST-SH-VERT, Q1 SI2301CDS, U1 REDBEAR_BLE_NANO2_LESS, U2 MCP73831T-2ACI/OT, U3 POLULU_DRV8835

Commit message: lkvfjkladsjf
Parts:
- BAT, PWR: value M02JST-SH-VERT -> M02JST-SH-RA; device a_parts:JST-2-SH-VERT -> a_parts:JST-2-SH-RA
- M1, M2: value M02JST-SH-VERT -> M02PTH-2MM; device a_parts:JST-2-SH-VERT -> a_parts:1X02-2MM-PTH
- moved C2 35.6 mm to (12.2, 42.0)
- moved U2 33.8 mm to (22.9, 34.7)
- moved R3 31.9 mm to (7.80, 33.9), turned to 0 degrees
- moved C1 30.7 mm to (5.30, 37.4), turned to 270 degrees
- moved CHARGE 24.5 mm to (25.1, 37.6), flipped to the top, turned to 270 degrees
- moved BAT 24.4 mm to (6.50, 29.5)
- moved R2 23.3 mm to (13.8, 31.4), turned to 0 degrees
- moved R1 22.6 mm to (16.0, 35.6), turned to 180 degrees
- moved D1 20.4 mm to (16.4, 27.0), flipped to the top, turned to 270 degrees
- moved M1 17.9 mm to (13.0, 2.00), turned to 180 degrees
- moved R4 17.2 mm to (20.2, 41.2), flipped to the bottom, turned to 270 degrees
- moved Q1 17.0 mm to (11.5, 27.0), flipped to the top, turned to 90 degrees
- moved M2 11.5 mm to (17.0, 2.00), turned to 180 degrees
- moved PWR 10.5 mm to (23.5, 29.5), flipped to the bottom, turned to 180 degrees
- moved U3 7.85 mm to (15.0, 15.0), flipped to the bottom
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Connections:
- net AIN1: now also U1.16; no longer U1.13
- net AIN2: now also U1.15; no longer U1.16
- net BIN1: now also U1.14; no longer U1.15
- net BIN2: now also U1.13; no longer U1.14
- net N$4: now also M1.P$2; no longer M1.2
- net N$5: now also M1.P$1; no longer M1.1
- net N$6: now also M2.P$2; no longer M2.2
- net N$7: now also M2.P$1; no longer M2.1
Other:
- board size 20 x 18 mm -> 30 x 30 mm
- board text removed: "AIN1"
- board text removed: "AIN2"
- board text removed: "BIN1"
- board text removed: "BIN2"
- board text removed: "GND"
- board text removed: "NC"
- board text removed: "USB PWR ONLY"
- board text removed: "VDD"
- board text removed: "VIN"
