File: hardware/maus-blenano2-mk-1.0.2.sch (EAGLE design)
At the start: 17 parts, among them M1 M02JST-SH-VERT, M2 M02JST-SH-VERT, Q1 SI2301CDS, U1 REDBEAR_BLE_NANO2_LESS, U2 MCP73831T-2ACI/OT, U3 POLULU_DRV8835

Commit message: lkvfjkladsjf
Parts:
- removed M1, M2: M02JST-SH-VERT, a_parts:M02JST-SH-VERT
- removed R4: 10K, a_parts:RESISTORR0603-TIGHTER
- removed U3: POLULU_DRV8835, a_parts:POLULU_DRV8835
- added JP1: (no value), a_parts:M07PTH-CENTERED
- BAT, PWR: value M02JST-SH-VERT -> M02JST-SH-RA; device a_parts:M02JST-SH-VERT -> a_parts:M02JST-SH-RA
- FRAME1: VERSION v1.1.0 -> v1.0.2
- renumbered CHARGE to CHG
Connections:
- removed net N$3: R4.2, U3.MODE
- removed net N$4: M1.2, U3.AO1
- removed net N$5: M1.1, U3.AO2
- removed net N$6: M2.2, U3.BO1
- removed net N$7: M2.1, U3.BO2
- net 3.3V: now also JP1.5; no longer R4.1, U3.VCC
- net 5V: now also D1.A1
- net AIN1: now also JP1.1, U1.D2; no longer U1.D3, U3.AIN1
- net AIN2: now also JP1.2, U1.D1; no longer U1.D2, U3.AIN2
- net BIN1: now also JP1.3, U1.D0; no longer U1.D1, U3.BIN1
- net BIN2: now also JP1.4, U1.D3; no longer U1.D0, U3.BIN2
- net GND: now also JP1.7; no longer U3.GND
- net VIN: now also JP1.6; no longer U3.VIN
Other:
- moved on the sheet: BAT, PWR
