File: hardware/maus-blenano2-mk-1.0.3.sch (EAGLE design)
At the start: 17 parts, among them M1 M02PTH-2MM, M2 M02PTH-2MM, Q1 SI2301CDS, U1 REDBEAR_BLE_NANO2_LESSSMD, U2 MCP73831T-2ACI/OT, U3 POLULU_DRV8835SMT_OUTER

Commit message: moar boards
Parts:
- removed R4: 10K, a_parts:RESISTORR0603-TIGHTER
- added C3: 2.2uF@25V, a_parts:CAPACITOR-CERAMICC0603
- added C4: 10nF@16V, a_parts:CAPACITOR-CERAMICC0402
- added C5: 22uF@16V, a_parts:CAPACITOR-CERAMICC1206
- C1, C2: value 4.7uF -> 4.7uF@16V
- FRAME1: VERSION v1.0.1 -> v1.0.3
- U1: value REDBEAR_BLE_NANO2_LESSSMD -> REDBEAR_BLE_NANO2_LESS; device a_parts:REDBEAR_BLE_NANO2_LESSSMD -> a_parts:REDBEAR_BLE_NANO2_LESS
- U3: value POLULU_DRV8835SMT_OUTER -> DRV8833; device a_parts:POLULU_DRV8835SMT_OUTER -> a_parts:DRV8833PW
- renumbered CHARGE to CHG
Connections:
- net N$4 renamed MA1
- net N$5 renamed MA2
- net N$6 renamed MB1
- net N$7 renamed MB2
- new net !SLEEP: U1.D3, U3.!SLEEP
- new net N$4: C4.1, U3.VCP
- net 3.3V: no longer R4.1, U3.VCC
- net 5V: now also D1.A1
- net AIN1: now also U1.D1; no longer U1.D2
- net AIN2: now also U1.D0; no longer U1.D1
- net BIN1: now also U1.D4; no longer U1.D0
- net BIN2: now also U1.D5; no longer U1.D3
- net GND: now also C3.2, C5.2, U3.ASENSE, U3.BSENSE
- net N$3: now also C3.1, U3.VINT; no longer R4.2, U3.MODE
- net VIN: now also C4.2, C5.1, U3.VM; no longer U3.VIN
Other:
- moved on the sheet: D1, M1, M2, Q1, R2
