File: hardware/maus-blenano2-mk-1.1.0.brd (EAGLE design)
At the start: 30 x 30 mm, 17 parts, among them M1 M02PTH-2MM, M2 M02PTH-2MM, Q1 SI2301CDS, U1 REDBEAR_BLE_NANO2_LESSSMD, U2 MCP73831T-2ACI/OT, U3 POLULU_DRV8835SMT_OUTER

Commit message: moar boards
Parts:
- removed CHARGE: LED0603-TIGHT, a_parts:LED-0603-TIGHT
- removed R4: 10K, a_parts:R0603-TIGHTER
- added C3: 2.2uF@25V, a_parts:C0603
- added C4: 10nF@16V, a_parts:C0402
- added C5: 22uF@16V, a_parts:C1206
- added CHG: LED0603-TIGHT, a_parts:LED-0603-TIGHT
- C1, C2: value 4.7uF -> 4.7uF@16V
- U1: value REDBEAR_BLE_NANO2_LESSSMD -> REDBEAR_BLE_NANO2_LESS; device a_parts:REDBEAR_BLE_NANO2_LESS_SMD -> a_parts:REDBEAR_BLE_NANO2_LESS
- U3: value POLULU_DRV8835SMT_OUTER -> DRV8833; device a_parts:POLULU_DRV8835_SMT_OUTER -> a_parts:TSSOP16
- moved R1 22.1 mm to (7.00, 9.50), flipped to the bottom, turned to 180 degrees
- moved R3 17.4 mm to (11.0, 9.50), flipped to the bottom, turned to 180 degrees
- moved C2 11.7 mm to (5.00, 12.5), flipped to the bottom, turned to 270 degrees
- moved M1 10.0 mm to (7.00, 1.50), turned to 180 degrees
- moved D1 9.60 mm to (11.0, 14.5), turned to 180 degrees
- moved Q1 9.60 mm to (7.00, 14.5), turned to 270 degrees
- moved PWR 8.28 mm to (15.0, 19.5)
- moved U3 7.81 mm to (9.00, 6.50), flipped to the top, turned to 0 degrees
- moved U1 6.71 mm to (9.00, 10.5), turned to 0 degrees
- moved U2 6.50 mm to (9.00, 12.5), flipped to the bottom, turned to 180 degrees
- moved BAT 5.70 mm to (3.00, 19.5)
- moved C1 2.24 mm to (13.0, 12.5), flipped to the bottom, turned to 270 degrees
- moved M2 2.06 mm to (11.0, 1.50)
- moved R2 1.00 mm to (11.0, 17.5), turned to 0 degrees
Connections:
- removed net N$5: M1.P$1, U3.10
- removed net N$6: M2.P$2, U3.11
- removed net N$7: M2.P$1, U3.12
- new net !SLEEP: U1.13, U3.1
- new net MA1: M1.P$2, U3.2
- new net MA2: M1.P$1, U3.4
- new net MB1: M2.P$2, U3.7
- new net MB2: M2.P$1, U3.5
- net 3.3V: no longer R4.1, U3.2
- net 5V: now also CHG.A, D1.1; no longer CHARGE.A
- net AIN1: now also U1.15, U3.16; no longer U1.16, U3.6
- net AIN2: now also U1.14, U3.15; no longer U1.15, U3.5
- net BIN1: now also U1.3, U3.9; no longer U1.14, U3.4
- net BIN2: now also U1.4, U3.10; no longer U1.13, U3.3
- net GND: now also C3.2, C5.2, U3.13, U3.3, U3.6; no longer U3.1, U3.14
- net N$2: now also CHG.C; no longer CHARGE.C
- net N$3: now also C3.1, U3.14; no longer R4.2, U3.7
- net N$4: now also C4.1, U3.11; no longer M1.P$2, U3.9
- net VIN: now also C4.2, C5.1, U3.12; no longer U3.13
Routing:
- net 5V: track 0.00 -> 21.9 mm, vias 0 -> 1
- net VIN: track 0.00 -> 20.1 mm, vias 0 -> 1
- net FOO: track 0.00 -> 12.9 mm
- net N$2: track 0.00 -> 12.7 mm, vias 0 -> 1
- net VBAT: track 0.00 -> 12.4 mm, vias 0 -> 1
- net BIN2: track 0.00 -> 8.17 mm
- net AIN2: track 0.00 -> 8.17 mm
- net BIN1: track 0.00 -> 6.65 mm
- net AIN1: track 0.00 -> 6.65 mm
- net !SLEEP: track 0.00 -> 6.58 mm
- net MA1: track 0.00 -> 2.89 mm
- net MB1: track 0.00 -> 2.89 mm
- net MB2: track 0.00 -> 2.48 mm
- net MA2: track 0.00 -> 2.48 mm
- net N$4: track 0.00 -> 2.42 mm
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Other:
- board size 30 x 30 mm -> 18 x 21 mm
- board text added: "SQUEAK"
