File: hardware/redmaus-ir-tx-amp-mk-1.2.sch (EAGLE design)
At the start: 13 parts, among them Q1 MMBT2222A, Q2 MMBT2222A, Q3 MMBT2222A, Q4 MMBT2222A

Commit message: moar boards
Parts:
- removed LED3, LED4: LED3MMX2MM-SIDE-SMD, a_parts:LED3MMX2MM-SIDE-SMD
- removed Q3, Q4: MMBT2222A, a_parts:TRANSISTOR_NPNMMBT2222A
- removed R4: 10R, a_parts:RESISTORR0603-TIGHTER
- LED1, LED2: value LED3MMX2MM-SIDE-SMD -> LED5MM_SHORTPADS; device a_parts:LED3MMX2MM-SIDE-SMD -> a_parts:LED5MM_SHORTPADS
Connections:
- removed net N$2: LED3.C, Q3.C
- removed net N$5: Q3.E, Q4.B, R4.2
- removed net N$6: LED3.A, LED4.C
- net DATA-AMP: no longer Q3.B, Q4.C
- net GND: no longer Q4.E, R4.1
- net VCC: no longer LED4.A
